Commit message: lidar link spawn corrected

File: src/rover_description/urdf/rover_description.urdf.xacro (robot description, xacro)
@@ -760,5 +760,5 @@
   <joint
     name="lidar_joint" type="fixed">
-    <origin xyz="0 0 0" rpy="1.57 1.57 1.57"/>
+    <origin xyz="0 0.2 0" rpy="1.57 0 0"/>
     <parent link="differential_bar"/>
     <child link="lidar_link"/>

Commit message: added lidar support

File: src/rover_description/urdf/rover_description.urdf.xacro (robot description, xacro)
@@ -7,9 +7,16 @@
   xmlns:xacro="http://www.ros.org/wiki/xacro">
   <xacro:include filename="$(find rover_description)/urdf/sensors.urdf.xacro"/>
+  <!-- Standard ROS base_link root frame (REP-103: X forward, Y left, Z up) -->
+  <link name="base_link" />
+  <joint name="base_link_to_chassis_joint" type="fixed">
+    <parent link="base_link" />
+    <child link="chassis" />
+    <origin xyz="-0.9725 0.8488 -1.09" rpy="-1.570796 0 -1.570796" />
+  </joint>
   <link
     name="chassis">
     <inertial>
       <origin
-        xyz="0.848856756174826 1.01936314005979 1.40233565202935"
+        xyz="0.848856756174826 -1.40233565202935 1.01936314005979"
         rpy="0 0 0" />
       <mass
@@ -19,7 +26,7 @@
         ixy="-2.16162888765699E-10"
         ixz="2.16817247419927E-10"
-        iyy="0.00486414098649309"
+        iyy="0.0215591824716579"
         iyz="-3.67475478322892E-06"
-        izz="0.0215591824716579" />
+        izz="0.00486414098649309" />
     </inertial>
     <visual>
@@ -89,5 +96,5 @@
   <joint
     name="rocker_to_chassis_left_joint"
-    type="continuous">
+    type="revolute">
     <origin
       xyz="0.57581 -1.3985 1.0289"
@@ -99,4 +106,6 @@
     <axis
       xyz="0 0 1" />
+    <limit lower="-0.4" upper="0.4" effort="100.0" velocity="1.0" />
+    <dynamics damping="8.0" friction="0.5" />
   </joint>
   <link
@@ -195,5 +204,5 @@
   <joint
     name="bogie_to_rocker_left_joint"
-    type="continuous">
+    type="revolute">
     <origin
       xyz="0.33299 -0.19225 -0.005"
@@ -205,4 +214,6 @@
     <axis
       xyz="0 0 1" />
+    <limit lower="-0.4" upper="0.4" effort="100.0" velocity="1.0" />
+    <dynamics damping="5.0" friction="0.5" />
   </joint>
   <link
@@ -407,5 +418,5 @@
   <joint
     name="rocker_to_chassis_right_joint"
-    type="continuous">
+    type="revolute">
     <origin
       xyz="0.97481 -1.3985 1.0291"
@@ -417,4 +428,6 @@
     <axis
       xyz="0 0 1" />
+    <limit lower="-0.4" upper="0.4" effort="100.0" velocity="1.0" />
+    <dynamics damping="8.0" friction="0.5" />
   </joint>
   <link
@@ -513,5 +526,5 @@
   <joint
     name="rocker_to_bogie_right_joint"
-    type="continuous">
+    type="revolute">
     <origin
       xyz="-0.33299 -0.19225 0"
@@ -523,4 +536,6 @@
     <axis
       xyz="0 0 1" />
+    <limit lower="-0.4" upper="0.4" effort="100.0" velocity="1.0" />
+    <dynamics damping="5.0" friction="0.5" />
   </joint>
   <link
@@ -733,26 +748,35 @@
     <child
       link="differential_bar" />
-    <axis
-      xyz="0 1 0" />
   </joint>
   <link name="lidar_link">
     <inertial>
-      <origin xyz="0 0 0.2" rpy="0 0 0"/>
+      <origin xyz="0 0 0" rpy="0 0 0"/>
       <mass value="0.1"/>
       <inertia ixx="0.0000658" ixy="0" ixz="0" iyy="0.0000658" iyz="0" izz="0.000125" />
     </inertial>
-    <visual>
-      <origin xyz="0 0 0.2" rpy="0 0 0"/>
-      <geometry>
-        <cylinder radius="0.05" length="0.02"/>
+    <!-- Sensor head visual -->
+    <visual>
+      <origin xyz="0 0 0" rpy="0 0 0"/>
+      <geometry>
+        <cylinder radius="0.05" length="0.04"/>
       </geometry>
       <material name="black">
-        <color rgba="0 0 0 1"/>
-      </material>
-    </visual>
-    <collision>
-      <origin xyz="0 0 0.2" rpy="0 0 0"/>
-      <geometry>
-        <cylinder radius="0.05" length="0.02"/>
+        <color rgba="0.1 0.1 0.1 1"/>
+      </material>
+    </visual>
+    <!-- Mount post/riser to differential bar -->
+    <visual name="lidar_mast">
+      <origin xyz="0 0 -0.08" rpy="0 0 0"/>
+      <geometry>
+        <cylinder radius="0.015" length="0.16"/>
+      </geometry>
+      <material name="dark_grey">
+        <color rgba="0.3 0.3 0.3 1"/>
+      </material>
+    </visual>
+    <collision>
+      <origin xyz="0 0 0" rpy="0 0 0"/>
+      <geometry>
+        <cylinder radius="0.05" length="0.04"/>
       </geometry>
     </collision>
@@ -760,5 +784,5 @@
   <joint
     name="lidar_joint" type="fixed">
-    <origin xyz="0 0.2 0" rpy="1.57 0 0"/>
+    <origin xyz="0 -0.16 0" rpy="1.570796 -1.550981 0"/>
     <parent link="differential_bar"/>
     <child link="lidar_link"/>
@@ -836,8 +860,33 @@
       <state_interface name="position" />
     </joint>
-    <joint name="differential_bar_to_chassis_joint">
-      <state_interface name="position" />
-    </joint>
   </ros2_control>
+  <!-- WHEEL FRICTION FOR GAZEBO -->
+  <gazebo reference="front_wheel_left"><mu1>1.2</mu1><mu2>1.2</mu2></gazebo>
+  <gazebo reference="middle_wheel_left"><mu1>1.2</mu1><mu2>1.2</mu2></gazebo>
+  <gazebo reference="back_wheel_left"><mu1>1.2</mu1><mu2>1.2</mu2></gazebo>
+  <gazebo reference="front_wheel_right"><mu1>1.2</mu1><mu2>1.2</mu2></gazebo>
+  <gazebo reference="middle_wheel_right"><mu1>1.2</mu1><mu2>1.2</mu2></gazebo>
+  <gazebo reference="back_wheel_right"><mu1>1.2</mu1><mu2>1.2</mu2></gazebo>
+  <!-- ROCKER-BOGIE SUSPENSION DYNAMICS & SPRINGS -->
+  <gazebo reference="rocker_to_chassis_left_joint">
+    <implicitSpringDamper>true</implicitSpringDamper>
+    <springStiffness>45.0</springStiffness>
+    <springReference>0.0</springReference>
+  </gazebo>
+  <gazebo reference="rocker_to_chassis_right_joint">
+    <implicitSpringDamper>true</implicitSpringDamper>
+    <springStiffness>45.0</springStiffness>
+    <springReference>0.0</springReference>
+  </gazebo>
+  <gazebo reference="bogie_to_rocker_left_joint">
+    <implicitSpringDamper>true</implicitSpringDamper>
+    <springStiffness>25.0</springStiffness>
+    <springReference>0.0</springReference>
+  </gazebo>
+  <gazebo reference="rocker_to_bogie_right_joint">
+    <implicitSpringDamper>true</implicitSpringDamper>
+    <springStiffness>25.0</springStiffness>
+    <springReference>0.0</springReference>
+  </gazebo>
   <gazebo>
     <plugin filename="gz_ros2_control-system" name="gz_ros2_control::GazeboSimROS2ControlPlugin">
@@ -845,3 +894,3 @@
     </plugin>
   </gazebo>
-  </robot>
+</robot>

File: src/rover_description/urdf/sensors.urdf.xacro (robot description, xacro)
@@ -33,3 +33,57 @@
     </sensor>
   </gazebo>
+  <!-- ========================================================= -->
+  <!--                          IMU                              -->
+  <!-- ========================================================= -->
+  <gazebo reference="chassis">
+    <sensor name="chassis_imu" type="imu">
+      <always_on>true</always_on>
+      <update_rate>100</update_rate>
+      <visualize>false</visualize>
+      <topic>/imu/data</topic>
+      <gz_frame_id>base_link</gz_frame_id>
+      <imu>
+        <angular_velocity>
+          <x>
+            <noise type="gaussian">
+              <mean>0.0</mean>
+              <stddev>0.001</stddev>
+            </noise>
+          </x>
+          <y>
+            <noise type="gaussian">
+              <mean>0.0</mean>
+              <stddev>0.001</stddev>
+            </noise>
+          </y>
+          <z>
+            <noise type="gaussian">
+              <mean>0.0</mean>
+              <stddev>0.001</stddev>
+            </noise>
+          </z>
+        </angular_velocity>
+        <linear_acceleration>
+          <x>
+            <noise type="gaussian">
+              <mean>0.0</mean>
+              <stddev>0.01</stddev>
+            </noise>
+          </x>
+          <y>
+            <noise type="gaussian">
+              <mean>0.0</mean>
+              <stddev>0.01</stddev>
+            </noise>
+          </y>
+          <z>
+            <noise type="gaussian">
+              <mean>0.0</mean>
+              <stddev>0.01</stddev>
+            </noise>
+          </z>
+        </linear_acceleration>
+      </imu>
+    </sensor>
+  </gazebo>
 </robot>
